Commit message: Rectified some errors in the urdf files and added controller for the movement of the bot.

File: urdf/accessories/kinect_camera.urdf.xacro (robot description, xacro)
@@ -34,5 +34,5 @@
         <origin xyz="0 0 0" rpy="0 0 ${M_PI/2}"/>
         <geometry>
-          <mesh filename="package://husky_description/meshes/accessories/kinect.dae" />
+          <mesh filename="package://husky_sim/meshes/accessories/kinect.dae" />
         </geometry>
       </visual>

File: urdf/accessories/sensor_arch.urdf.xacro (robot description, xacro)
@@ -7,5 +7,5 @@
              <visual>
                  <geometry>
-                     <mesh filename="package://husky_description/meshes/accessories/${size}_mm_sensor_arch.dae" />
+                     <mesh filename="package://husky_sim/meshes/accessories/${size}_mm_sensor_arch.dae" />
                  </geometry>
              </visual>
@@ -13,5 +13,5 @@
                  <origin xyz="0 0 0" rpy="0 0 0"/>
                  <geometry>
-                     <mesh filename="package://husky_description/meshes/accessories/${size}_mm_sensor_arch.dae" />
+                     <mesh filename="package://husky_sim/meshes/accessories/${size}_mm_sensor_arch.dae" />
                  </geometry>
              </collision>

File: urdf/accessories/sick_lms1xx_mount.urdf.xacro (robot description, xacro)
@@ -33,5 +33,5 @@
         <geometry>
           <!-- Origin of this mesh is the base of the bracket. -->
-          <mesh filename="package://husky_description/meshes/accessories/lms1xx_mount.dae" />
+          <mesh filename="package://husky_sim/meshes/accessories/lms1xx_mount.dae" />
         </geometry>
       </visual>

File: urdf/decorations.urdf.xacro (robot description, xacro)
@@ -30,5 +30,5 @@
         <origin xyz="0 0 0" rpy="0 0 0" />
         <geometry>
-          <mesh filename="package://husky_description/meshes/top_chassis.dae" />
+          <mesh filename="package://husky_sim/meshes/top_chassis.dae" />
         </geometry>
       </visual>
@@ -44,5 +44,5 @@
         <visual>
           <geometry>
-            <mesh filename="package://husky_description/meshes/user_rail.dae" />
+            <mesh filename="package://husky_sim/meshes/user_rail.dae" />
           </geometry>
         </visual>
@@ -59,5 +59,5 @@
       <visual>
         <geometry>
-          <mesh filename="package://husky_description/meshes/bumper.dae" />
+          <mesh filename="package://husky_sim/meshes/bumper.dae" />
         </geometry>
       </visual>
@@ -73,5 +73,5 @@
           <visual>
               <geometry>
-                  <mesh filename="package://husky_description/meshes/bumper_extension.dae" />
+                  <mesh filename="package://husky_sim/meshes/bumper_extension.dae" />
               </geometry>
           </visual>
@@ -87,5 +87,5 @@
       <visual>
         <geometry>
-          <mesh filename="package://husky_description/meshes/bumper.dae" />
+          <mesh filename="package://husky_sim/meshes/bumper.dae" />
         </geometry>
       </visual>
@@ -101,5 +101,5 @@
           <visual>
               <geometry>
-                  <mesh filename="package://husky_description/meshes/bumper_extension.dae" />
+                  <mesh filename="package://husky_sim/meshes/bumper_extension.dae" />
               </geometry>
           </visual>
@@ -118,5 +118,5 @@
             <origin xyz="0 0 0" rpy="0 0 0" />
             <geometry>
-              <mesh filename="package://husky_description/meshes/large_top_plate.dae" />
+              <mesh filename="package://husky_sim/meshes/large_top_plate.dae" />
             </geometry>
           </visual>
@@ -124,5 +124,5 @@
             <origin xyz="0 0 0" rpy="0 0 0"/>
             <geometry>
-              <mesh filename="package://husky_description/meshes/large_top_plate_collision.stl" />
+              <mesh filename="package://husky_sim/meshes/large_top_plate_collision.stl" />
             </geometry>
           </collision>
@@ -152,5 +152,5 @@
             <origin xyz="0 0 0" rpy="0 0 0" />
             <geometry>
-              <mesh filename="package://husky_description/meshes/top_plate.dae" />
+              <mesh filename="package://husky_sim/meshes/top_plate.dae" />
             </geometry>
           </visual>
@@ -158,5 +158,5 @@
             <origin xyz="0 0 0" rpy="0 0 0"/>
             <geometry>
-              <mesh filename="package://husky_description/meshes/top_plate.stl" />
+              <mesh filename="package://husky_sim/meshes/top_plate.stl" />
             </geometry>
           </collision>

File: urdf/husky.urdf.xacro (robot description, xacro)
@@ -31,11 +31,11 @@
   <xacro:property name="husky_rear_bumper_extend" value="$(optenv HUSKY_REAR_BUMPER_EXTEND 0)" />
   <xacro:arg name="robot_namespace" default="/" />
-  <xacro:arg name="urdf_extras" default="empty.urdf" />
+  <!-- <xacro:arg name="urdf_extras" default="empty.urdf" /> -->
   <!-- Included URDF/XACRO Files -->
-  <xacro:include filename="$(find husky_description)/urdf/decorations.urdf.xacro" />
-  <xacro:include filename="$(find husky_description)/urdf/wheel.urdf.xacro" />
-  <xacro:include filename="$(find husky_description)/urdf/accessories/kinect_camera.urdf.xacro"/>
-  <xacro:include filename="$(find husky_description)/urdf/accessories/sick_lms1xx_mount.urdf.xacro"/>
-  <xacro:include filename="$(find husky_description)/urdf/accessories/sensor_arch.urdf.xacro"/>
+  <xacro:include filename="$(find husky_sim)/urdf/decorations.urdf.xacro" />
+  <xacro:include filename="$(find husky_sim)/urdf/wheel.urdf.xacro" />
+  <xacro:include filename="$(find husky_sim)/urdf/accessories/kinect_camera.urdf.xacro"/>
+  <xacro:include filename="$(find husky_sim)/urdf/accessories/sick_lms1xx_mount.urdf.xacro"/>
+  <xacro:include filename="$(find husky_sim)/urdf/accessories/sensor_arch.urdf.xacro"/>
   <xacro:property name="M_PI" value="3.14159"/>
   <!-- Base Size -->
@@ -55,5 +55,5 @@
       <origin xyz="0 0 0" rpy="0 0 0" />
       <geometry>
-        <mesh filename="package://husky_description/meshes/base_link.dae" />
+        <mesh filename="package://husky_sim/meshes/base_link.dae" />
       </geometry>
     </visual>
@@ -169,5 +169,21 @@
     </plugin>
   </gazebo>
+  <gazebo>
+    <plugin name="husky_controller" filename="libgazebo_ros_skid_steer_drive.so">
+	<updateRate>100.0</updateRate>
+	<robotNamespace>/</robotNamespace>
+	<leftFrontJoint>front_left_wheel</leftFrontJoint>
+	<rightFrontJoint>front_right_wheel</rightFrontJoint>
+	<leftRearJoint>rear_left_wheel</leftRearJoint>
+	<rightRearJoint>rear_right_wheel</rightRearJoint>
+	<wheelSeparation>0.556</wheelSeparation>
+	<wheelDiameter>0.330</wheelDiameter>
+	<robotBaseFrame>base_link</robotBaseFrame>
+	<torque>1</torque>
+	<topicName>cmd_vel</topicName>
+	<broadcastTF>0</broadcastTF>
+    </plugin>
+  </gazebo>
   <!-- Optional custom includes. -->
-  <xacro:include filename="$(arg urdf_extras)" />
+ <!-- <xacro:include filename="$(arg urdf_extras)" />  -->
 </robot>

File: urdf/wheel.urdf.xacro (robot description, xacro)
@@ -32,5 +32,5 @@
 				<origin xyz="0 0 0" rpy="0 0 0" />
 				<geometry>
-					<mesh filename="package://husky_description/meshes/wheel.dae" />
+					<mesh filename="package://husky_sim/meshes/wheel.dae" />
 				</geometry>
 			</visual>
